File: snac/SNAC  7ch SNES in Housing - Compact.sch (EAGLE design)
At the start: 10 parts, among them U1 PMIC-LDO-XC6206P332MR-G(SOT23), X2 JST-XH-09-PIN-LONG-PAD

Commit message: Add Compact SNES version, and WIP SNES Multitap
Parts:
- removed JP1, JP2: PINHD-1X10_2.54-S, pinhead-2:PINHD-1X10_2.54-S
Connections:
- net GND: no longer JP1.6, JP2.6
- net HV: no longer JP2.5
- net HV1: no longer JP2.1
- net HV2: no longer JP2.2
- net HV3: no longer JP2.3
- net HV4: no longer JP2.4
- net HV5: no longer JP2.7
- net HV6: no longer JP2.8
- net HV7: no longer JP2.9
- net HV8: no longer JP2.10
- net LV: no longer JP1.5
- net LV1: no longer JP1.1
- net LV2: no longer JP1.2
- net LV3: no longer JP1.3
- net LV4: no longer JP1.4
- net LV5: no longer JP1.7
- net LV6: no longer JP1.8
- net LV7: no longer JP1.9
- net LV8: no longer JP1.10
Other:
- note removed: "High Voltage"
- note removed: "Low Voltage"
