File: snac/SNAC  7ch SMS 3D Dongle.brd (EAGLE design)
At the start: 37.2 x 21.9 mm, 11 parts, among them IC1 4030D, K2 692112030100, Q9 BC849SMD, X2 STEREOJACK

Commit message: removed the Compact, TXS chip, and SMS3D with USB3 plug versions
Connections:
- net LV5: no longer R20.1
- net LV6: now also R20.1
Routing:
- net LV5: track 23.6 -> 0.00 mm, vias 2 -> 0
- net LV6: track 0.06 -> 22.6 mm, vias 0 -> 2
Changed lines of the file:
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@@
 <setting verticaltext="up"/>
 </settings>
-<grid distance="3" unitdist="mil" unit="mm" style="lines" multiple="1" display="no" altdistance="0.001" altunitdist="inch" altunit="inch"/>
+<grid distance="3" unitdist="mil" unit="mil" style="lines" multiple="1" display="no" altdistance="0.001" altunitdist="inch" altunit="inch"/>
 <layers>
 <layer number="1" name="Top" color="4" fill="1" visible="yes" active="yes"/>
@@
 <layer number="128" name="_bValues" color="7" fill="1" visible="no" active="no"/>
 <layer number="129" name="Mask" color="7" fill="1" visible="no" active="no"/>
+<layer number="130" name="SMDSTROOK" color="7" fill="1" visible="yes" active="yes"/>
 <layer number="131" name="tAdjust" color="7" fill="1" visible="no" active="no"/>
 <layer number="132" name="bAdjust" color="7" fill="1" visible="no" active="no"/>
+<layer number="133" name="mtFinish" color="7" fill="1" visible="yes" active="yes"/>
+<layer number="134" name="mbFinish" color="7" fill="1" visible="yes" active="yes"/>
+<layer number="135" name="mtGlue" color="7" fill="1" visible="yes" active="yes"/>
+<layer number="136" name="mbGlue" color="7" fill="1" visible="yes" active="yes"/>
+<layer number="137" name="mtTest" color="7" fill="1" visible="yes" active="yes"/>
+<layer number="138" name="mbTest" color="7" fill="1" visible="yes" active="yes"/>
+<layer number="139" name="mtKeepout" color="7" fill="1" visible="yes" active="yes"/>
+<layer number="140" name="mbKeepout" color="7" fill="1" visible="yes" active="yes"/>
+<layer number="141" name="mtRestrict" color="7" fill="1" visible="yes" active="yes"/>
+<layer number="142" name="mbRestrict" color="7" fill="1" visible="yes" active="yes"/>
+<layer number="143" name="mvRestrict" color="7" fill="1" visible="yes" active="yes"/>
 <layer number="144" name="Drill_legend" color="7" fill="1" visible="no" active="yes"/>
+<layer number="145" name="mHoles" color="7" fill="1" visible="yes" active="yes"/>
+<layer number="146" name="mMilling" color="7" fill="1" visible="yes" active="yes"/>
+<layer number="147" name="mMeasures" color="7" fill="1" visible="yes" active="yes"/>
+<layer number="148" name="mDocument" color="7" fill="1" visible="yes" active="yes"/>
+<layer number="149" name="mReference" color="7" fill="1" visible="yes" active="yes"/>
 <layer number="150" name="Notes" color="7" fill="1" visible="no" active="no"/>
 <layer number="151" name="HeatSink" color="7" fill="1" visible="no" active="yes"/>
@@
 <layer number="154" name="FabDoc2" color="7" fill="1" visible="no" active="no"/>
 <layer number="155" name="FabDoc3" color="7" fill="1" visible="no" active="no"/>
+<layer number="191" name="mNets" color="7" fill="1" visible="yes" active="yes"/>
+<layer number="192" name="mBusses" color="7" fill="1" visible="yes" active="yes"/>
+<layer number="193" name="mPins" color="7" fill="1" visible="yes" active="yes"/>
+<layer number="194" name="mSymbols" color="7" fill="1" visible="yes" active="yes"/>
+<layer number="195" name="mNames" color="7" fill="1" visible="yes" active="yes"/>
+<layer number="196" name="mValues" color="7" fill="1" visible="yes" active="yes"/>
 <layer number="199" name="Contour" color="7" fill="1" visible="no" active="yes"/>
 <layer number="200" name="200bmp" color="1" fill="10" visible="no" active="no"/>
@@
 <signal name="LV5">
 <contactref element="K2" pad="6"/>
-<wire x1="5.08" y1="12.7" x2="5.08" y2="12.668" width="0.1778" layer="1"/>
-<contactref element="R20" pad="1"/>
-<wire x1="24.3586" y1="16.725" x2="24.3586" y2="17.78" width="0.4064" layer="1"/>
-<wire x1="24.3586" y1="17.78" x2="24.1554" y2="17.9832" width="0.4064" layer="1"/>
-<via x="24.1554" y="17.9832" extent="1-16" drill="0.35"/>
-<wire x1="24.1554" y1="17.9832" x2="10.7442" y2="17.9832" width="0.4064" layer="16"/>
-<wire x1="7.7724" y1="15.0114" x2="7.7724" y2="13.335" width="0.4064" layer="16"/>
-<via x="7.7724" y="13.335" extent="1-16" drill="0.35"/>
-<wire x1="7.7724" y1="13.335" x2="7.1374" y2="12.7" width="0.4064" layer="1"/>
-<wire x1="7.1374" y1="12.7" x2="5.08" y2="12.7" width="0.4064" layer="1"/>
-<wire x1="10.7442" y1="17.9832" x2="7.7724" y2="15.0114" width="0.4064" layer="16"/>
 </signal>
 <signal name="LV6">
 <contactref element="K2" pad="5"/>
 <wire x1="5.08" y1="14.732" x2="5.08" y2="14.668" width="0.1778" layer="1"/>
+<contactref element="R20" pad="1"/>
+<wire x1="24.3586" y1="16.725" x2="24.3586" y2="17.78" width="0.4064" layer="1"/>
+<wire x1="24.3586" y1="17.78" x2="24.1554" y2="17.9832" width="0.4064" layer="1"/>
+<via x="24.1554" y="17.9832" extent="1-16" drill="0.3302"/>
+<wire x1="24.1554" y1="17.9832" x2="23.241" y2="18.8976" width="0.4064" layer="16"/>
+<wire x1="23.241" y1="18.8976" x2="10.1346" y2="18.8976" width="0.4064" layer="16"/>
+<wire x1="10.1346" y1="18.8976" x2="7.0866" y2="15.8496" width="0.4064" layer="16"/>
+<via x="7.0866" y="15.8496" extent="1-16" drill="0.3302"/>
+<wire x1="7.0866" y1="15.8496" x2="6.1976" y2="15.8496" width="0.4064" layer="1"/>
+<wire x1="6.1976" y1="15.8496" x2="5.08" y2="14.732" width="0.4064" layer="1"/>
 </signal>
 <signal name="LV7">
